File: FlippyAdapter.kicad_sch (KiCad schematic)
At the start: 3 parts, among them J1 Conn_02x20_Odd_Even, J2 Conn_02x20_Odd_Even, J3 Board Harness

Commit message: Add libraries submodule
Parts:
- J3: footprint FlippyAdapter:Connector_MegaMax_3000 -> Nieto_Connector:Luminator_MAX3000; symbol Connector_Generic:Conn_02x32_Odd_Even -> Nieto_Connector:Luminator_MAX3000
Changed lines of the file:
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@@
     (pin "1")
   )
-  (symbol (lib_id "Connector_Generic:Conn_02x32_Odd_Even") (at 106.045 99.695 0) (unit 1)
+  (symbol (lib_id "Nieto_Connector:Luminator_MAX3000") (at 106.045 99.695 0) (unit 1)
     (in_bom yes) (on_board yes)
     (property "Reference" "J3" (id 0) (at 107.315 56.0832 0))
     (property "Value" "Board Harness" (id 1) (at 107.315 58.3946 0))
-    (property "Footprint" "FlippyAdapter:Connector_MegaMax_3000" (id 2) (at 106.045 99.695 0)
+    (property "Footprint" "Nieto_Connector:Luminator_MAX3000" (id 2) (at 106.045 99.695 0)
       (effects (font (size 1.27 1.27)) hide)
     )
@@
     )
     (path "/7d3437a4-c2c3-479e-b868-7ec58b2519f5"
-      (reference "J3") (unit 1) (value "Board Harness") (footprint "FlippyAdapter:Connector_MegaMax_3000")
+      (reference "J3") (unit 1) (value "Board Harness") (footprint "Nieto_Connector:Luminator_MAX3000")
     )
   )
